Commit message: fix

File: cartographer_ros/cartographer_ros/urdf/fd_base.urdf (robot description, URDF)
Before this commit: robot cartographer_fd_base, 3 links, 2 joints
Joints:
- joint imu_link_joint: origin xyz=0.15 0 0.02 rpy=0 0 0.7854 -> xyz=0.15 0 0.02 rpy=0 0 -1.57
- joint laser_link_joint: origin xyz=0.15 0 0.0558 rpy=0 0 -0.7854 -> xyz=0.15 0 0.0558 rpy=0 0 1.57

Commit message: fix

File: cartographer_ros/cartographer_ros/urdf/fd_base.urdf (robot description, URDF)
Before this commit: robot cartographer_fd_base, 3 links, 2 joints
Joints:
- joint imu_link_joint: origin xyz=0 0 0 -> xyz=0.15 0 0.02 rpy=0 0 0.7854
- joint laser_link_joint: origin xyz=0 0 0 rpy=0 0 0 -> xyz=0.15 0 0.0558 rpy=0 0 -0.7854

Commit message: add realsense

File: cartographer_ros/cartographer_ros/urdf/fd_base.urdf (robot description, URDF)
Before this commit: robot lio, 4 links, 3 joints
Links:
- added link camera_left_depth_optical_frame
- added link camera_right_depth_optical_frame
Joints:
- removed joint laser_joint
- added joint camera_left_joint: type fixed, parent base_link, child camera_left_depth_optical_frame, origin xyz=0.266842719249179 0.0881830869392123 0.0807512430601606 rpy=-2.00712863979348 0 -1.13446401379631
- added joint camera_right_joint: type fixed, parent base_link, child camera_right_depth_optical_frame, origin xyz=0.287973632336214 -0.0428676975873733 0.0807512430601605 rpy=-2.00712863979348 0 -2.00712863979348
- added joint lidar_joint: type fixed, parent base_link, child laser_link, origin xyz=0.15 0 0.1 rpy=0 0 0

File: nav2_bringup/urdf/fd_base.xacro (robot description, xacro)
@@ -9,8 +9,8 @@
     <origin xyz="0 0 0" rpy="0 0 0" />
   </joint>
-  <link name="livox_frame"> </link>
+  <link name="laser_link"> </link>
   <joint name="lidar_joint" type="fixed">
     <parent link="base_link" />
-    <child link="livox_frame" />
+    <child link="laser_link" />
     <origin xyz="0.15 0 0.1" rpy="0 0 0" />
   </joint>

Commit message: fix

File: cartographer_ros/cartographer_ros/urdf/fd_base.urdf (robot description, URDF)
Before this commit: robot lio, 6 links, 5 joints
Links:
- added link imu_link
Joints:
- added joint imu_joint: type fixed, parent base_link, child imu_link, origin xyz=0.12 -0.05 0.06 rpy=0 0 0

File: nav2_bringup/urdf/fd_base.xacro (robot description, xacro)
@@ -14,4 +14,10 @@
     <child link="laser_link" />
     <origin xyz="0.15 0 0.1" rpy="0 0 0" />
+  </joint>
+  <link name="imu_link"> </link>
+    <joint name="imu_joint" type="fixed">
+      <parent link="base_link" />
+      <child link="imu_link" />
+      <origin xyz="0.12 -0.05 0.06" rpy="0 0 0" />
   </joint>
   <link name="camera_left_depth_optical_frame"> </link>

Commit message: fix

File: cartographer_ros/cartographer_ros/urdf/fd_base.urdf (robot description, URDF)
Before this commit: robot lio, 7 links, 6 joints
Joints:
- joint camera_left_joint: origin xyz=0.266842719249179 0.0881830869392123 0.0807512430601606 rpy=-2.00712863979348 0 -1.13446401379631 -> xyz=0.25032 0.13367 0.07824 rpy=-1.5708 0 -1.134
- joint camera_right_joint: origin xyz=0.287973632336214 -0.0428676975873733 0.0807512430601605 rpy=-2.00712863979348 0 -2.00712863979348 -> xyz=0.28567 -0.098316 0.07824 rpy=-1.5708 0 -2.06
- joint lidar_joint: origin xyz=0.15 0 0.1 rpy=0 0 0 -> xyz=0.17 0 0.22 rpy=0 0 0

File: nav2_bringup/urdf/fd_base.xacro (robot description, xacro)
@@ -13,5 +13,5 @@
     <parent link="base_link" />
     <child link="laser_link" />
-    <origin xyz="0.15 0 0.1" rpy="0 0 0" />
+    <origin xyz="0.17 0 0.22" rpy="0 0 0" />
   </joint>
   <link name="imu_link"> </link>
@@ -25,6 +25,10 @@
     <parent link="base_link" />
     <child link="camera_left_depth_optical_frame" />
-    <origin xyz="0.266842719249179 0.0881830869392123 0.0807512430601606"
-            rpy="-2.00712863979348 0 -1.13446401379631" />
+    <!-- <origin xyz="0.256842719249179 0.1081830869392123 0.1607512430601606"  -->
+            <!-- rpy="-2.00712863979348 0 -1.13446401379631" /> -->
+    <!-- <origin xyz="0.25032 0.13367 0.07824"
+            rpy="-1.2043 0 -0.7854" /> -->
+    <origin xyz="0.25032 0.13367 0.07824"
+            rpy="-1.5708 0 -1.134" />
   </joint>
   <link name="camera_right_depth_optical_frame"> </link>
@@ -32,6 +36,10 @@
       <parent link="base_link" />
       <child link="camera_right_depth_optical_frame" />
-      <origin xyz="0.287973632336214 -0.0428676975873733 0.0807512430601605"
-              rpy="-2.00712863979348 0 -2.00712863979348" />
+      <!-- <origin xyz="0.277973632336214 -0.0628676975873733 0.1607512430601605"  -->
+              <!-- rpy="-2.00712863979348 0 -2.00712863979348" /> -->
+      <!-- <origin xyz="0.28567 -0.098316 0.07824"
+              rpy="-1.2043 0 -2.3562" /> -->
+      <origin xyz="0.28567 -0.098316 0.07824"
+              rpy="-1.5708 0 -2.06" />
     </joint>
   <link name="navsat_link"> </link>

Commit message: fix

File: cartographer_ros/cartographer_ros/urdf/fd_base.urdf (robot description, URDF)
Before this commit: robot lio, 7 links, 6 joints
Joints:
- joint camera_left_joint: origin xyz=0.25032 0.13367 0.07824 rpy=-1.5708 0 -1.134 -> xyz=0.3097 0.1142 0.062 rpy=-1.5708 0 -1.3304
- joint camera_right_joint: origin xyz=0.28567 -0.098316 0.07824 rpy=-1.5708 0 -2.06 -> xyz=0.3097 -0.1142 0.062 rpy=1.5708 0 1.3304

File: nav2_bringup/urdf/fd_base.xacro (robot description, xacro)
@@ -29,6 +29,6 @@
     <!-- <origin xyz="0.25032 0.13367 0.07824"
             rpy="-1.2043 0 -0.7854" /> -->
-    <origin xyz="0.25032 0.13367 0.07824"
-            rpy="-1.5708 0 -1.134" />
+    <origin xyz="0.3097 0.1142 0.062"
+            rpy="-1.5708 0 -1.3304" />
   </joint>
   <link name="camera_right_depth_optical_frame"> </link>
@@ -40,6 +40,6 @@
       <!-- <origin xyz="0.28567 -0.098316 0.07824"
               rpy="-1.2043 0 -2.3562" /> -->
-      <origin xyz="0.28567 -0.098316 0.07824"
-              rpy="-1.5708 0 -2.06" />
+      <origin xyz="0.3097 -0.1142 0.062"
+            rpy="1.5708 0 1.3304" />
     </joint>
   <link name="navsat_link"> </link>
